File: MarkIIIA/WiFi_12_14_2017/WiFi_Board/revisions/R1_1_0/WiFi_Board_R1_1_0.sch (EAGLE design)
At the start: 30 parts, among them P3 USB-B1HSB6, P4 POWER_JACKPTH, P9 44764-1201, U2 FT232RL

Commit message: Revise WiFi Board to increase Case Clearance
Parts:
- removed C7: 100nF, PatternAgents-ProtoPads:CAP0402-CAP
- removed P9: 44764-1201, nsvr:44764-1201
- removed U2: FT232RL, ftdichip-3:FT232RL
- added LED1: (no value), led:LEDCHIP-LED0603
- added P2: USB-B1HSB6, USB-B1HSB6:USB-B1HSB6
- BOOT, RST: value SW-TACTILE-PTS840P -> (none); device we-switch:SW-TACTILE-PTS840P -> PatternAgents-ProtoPads:JMP-2-NO-PTH
- C1: value 0.1uF -> 100n; device PatternAgents-ProtoPads:CAP0603-CAP -> PatternAgents-ProtoPads:CAP0402-CAP
- C2, C4: value 10uF -> 1uF; device PatternAgents-ProtoPads:CAP0603-CAP -> PatternAgents-ProtoPads:CAP0402-CAP
- C3: value 10uF -> 47u; device PatternAgents-ProtoPads:CAP0603-CAP -> SparkFun-Capacitors:CAP_POLD
- C5: value 10uF -> 0.1uF; device PatternAgents-ProtoPads:CAP0603-CAP -> PatternAgents-ProtoPads:CAP0402-CAP
- C6: value 100n -> 1uF; device we-rcl:CAPACITOR-0402 -> PatternAgents-ProtoPads:CAP0402-CAP
- P3: value USB-B1HSB6 -> 44764-1201; device USB-B1HSB6:USB-B1HSB6 -> nsvr:44764-1201
- R1, R3: value 4k7 -> 10k; device we-rcl:RESISTOR-0402 -> PatternAgents-ProtoPads:RESISTOR0402-TYP
- R10, R2: device we-rcl:RESISTOR-0402 -> PatternAgents-ProtoPads:RESISTOR0402-TYP
- R11, R9: value 10k -> 4k7; device we-rcl:RESISTOR-0402 -> PatternAgents-ProtoPads:RESISTOR0402-TYP
- R4: value 10k -> 220
- R5: value 10k -> 1k; device we-rcl:RESISTOR-0402 -> PatternAgents-ProtoPads:RESISTOR0402-TYP
- R6, R8: value 220 -> 10k; device we-rcl:RESISTOR-0402 -> PatternAgents-ProtoPads:RESISTOR0402-TYP
- R7: value 10k -> 220; device we-rcl:RESISTOR-0402 -> PatternAgents-ProtoPads:RESISTOR0402-TYP
- renumbered ESP8266 to ESP1, P4 to P1
Connections:
- removed net !PWREN_FTDI: R4.1, U2.CBUS3
- removed net !RXLED_FTDI: U2.CBUS1
- removed net !SLEEP_FTDI: U2.CBUS4
- removed net !TXDEN_FTDI: U2.CBUS2
- removed net !TXLED_FTDI: U2.CBUS0
- removed net 3V3_FTDI: C7.1, U2.3V3OUT
- removed net CTS_FTDI: U2._CTS
- removed net DCD_FTDI: U2._DCD
- removed net DSR_FTDI: U2._DSR
- removed net DTR_FTDI: U2._DTR
- removed net IO12: ESP1.MISO/IO12
- removed net IO14: ESP1.SCK/IO14
- removed net OSCI_FTDI: U2.OSCI
- removed net OSCO_FTDI: U2.OSCO
- removed net RI_FTDI: U2._RI
- removed net RTS_FTDI: U2._RTS
- removed net RXD_FTDI: U2.RXD
- removed net TXD_FTDI: U2.TXD
- removed net VDD: R4.2, U2.VCCIO
- new net LED1: LED1.A, R5.2
- net !RST: now also R7.1, R8.1; no longer R2.1, R5.1, U2._RESET
- net 3V3_EXT: now also C1.2, C3.+, C4.1, C5.1, P3.5, R11.2, R2.2, R8.2; no longer C1.1, C2.1, C3.1, C6.2, P9.5, R10.2, R5.2, R7.2
- net 5V0: now also P3.4; no longer P9.4, U2.VCC
- net CTS0: now also ESP1.MISO/IO12, P3.10; no longer P9.10
- net EN: now also R1.1; no longer R9.1
- net GND: now also BOOT.2, C1.1, C3.-, C6.2, LED1.C, P2.GND, P3.3, R10.1, RST.2; no longer BOOT.S1, C1.2, C3.2, C6.1, C7.2, P3.GND, P9.3, R11.1, RST.S1, U2.AGND, U2.GND1, U2.GND2, U2.GND3, U2.TEST
- net I2C_SCL: now also P3.6, R9.1; no longer P9.6, R3.1
- net I2C_SDA: now also P3.12, R11.1; no longer P9.12, R1.1
- net IO0: now also R3.1, R4.1, R5.1; no longer R7.1, R8.1
- net IO15: now also R10.2; no longer R11.2
- net IO16: now also R6.2; no longer R2.2
- net IO2: now also R2.1; no longer R10.1
- net N$1: now also R7.2, RST.1; no longer R6.2, RST.P1
- net N$2: now also BOOT.1, R4.2; no longer BOOT.P1, R8.2
- net RTS0: now also ESP1.SCK/IO14, P3.11; no longer P9.11
- net RXD0: now also P3.8; no longer P9.8
- net TXD0: now also P3.9; no longer P9.9
- net USB_DM: now also P2.D-, P3.7; no longer P3.D-, P9.7, U2.USBDM
- net USB_DP: now also P2.D+, P3.1; no longer P3.D+, P9.1, U2.USBDP
- net VBAT_DC: now also C6.1; no longer C5.1
- net VBUS_IN: now also P2.VCC; no longer P3.VCC
- net VIN: now also P3.2; no longer P9.2
- net VIN_DC: now also C2.1; no longer C4.1
Other:
- note added: "@Copyright 2018 NSVR All Rights Reserved Confidential and Proprietary Information"
- note added: "NSVR - ESP8266 Wi-Fi Board"
- note removed: "@Copyright 2016/2017 NSVR All Rights Reserved Confidential and Proprietary Information"
- note removed: "NSVR - BLTE Board"
- moved on the sheet: C1, C2, C4, C5, R4
