File: MarkIIIB/wifi_03_12_2018/wifi_03_12_2018.sch (EAGLE design)
At the start: 29 parts, among them P1 POWER_JACKPTH, P2 USB-B1HSB6, P3 44764-1201

Commit message: 03_12_2018 Update
Parts:
- renumbered C1 to C801, C2 to C802, C3 to C803, C4 to C804, C5 to C805, C6 to C806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
