File: MarkIIIB/wifi_03_12_2018/wifi_03_12_2018.brd (EAGLE design)
At the start: 51.8 x 43.2 mm, 29 parts, among them P1 POWER_JACKPTH, P2 USB-B1HSB6, P3 44764-1201

Commit message: 03_12_2018 Update
Parts:
- removed R2, R3: 10k, PatternAgents-ProtoPads:EIA-0402
- added R802, R803: 10k, PatternAgents-ProtoPads:EIA-0402
- renumbered C1 to C801, C2 to C802, C3 to C803, C4 to C804, C5 to C805, C6 to C806, D1 to D801, D2 to D802, ESP1 to U801, F1 to F801, LED1 to D803, P1 to P801, P2 to P802, P3 to P803, R1 to R801, R10 to R810, R11 to R811, R4 to R804, R5 to R805, R6 to R806, R7 to R807, R8 to R808, R9 to R809
Connections:
- net 3V3_EXT: now also R802.2, R803.2; no longer R2.2, R3.2
- net IO0: now also R803.1; no longer R3.1
- net IO2: now also R802.1; no longer R2.1
Other:
- board text added: "03/12/2018"
- board text added: "F801"
- board text removed: "1/24/2018"
- board text removed: "F1"

Commit message: Notch Wifi board for case clearances
Routing:
- net GND: track 275.1 -> 266.2 mm
- net I2C_SDA: track 38.7 -> 36.5 mm, vias 1 -> 2
Other:
- outline, holes or cut-outs redrawn
- board text added: "03/14/2018"
- board text added: "Rev. 1.1.1"
- board text removed: "03/12/2018"
- board text removed: "Rev. 1.1.0"
