File: MarkIIIB/driver_03_12_2018/driver_03_12_2018.brd (EAGLE design)
At the start: 27.9 x 43.9 mm, 40 parts, among them P201 503148-1690, P202 502494-0670, U201 PCA9548A_PW_24

Commit message: Add Part Number ROllup Spreadsheets
Parts:
- renumbered R19 to R219
Changed lines of the file:
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@@
 <element name="R217" library="resistor" package="R0402" value="10k" x="42.926" y="77.0382" smashed="yes"/>
 <element name="R218" library="PatternAgents-ProtoPads" package="EIA-0402" value="10k" x="50.69966875" y="75.058778125" smashed="yes" rot="R180"/>
-<element name="R19" library="PatternAgents-ProtoPads" package="EIA-0402" value="10k" x="53.87009375" y="75.058778125" smashed="yes" rot="R180"/>
+<element name="R219" library="PatternAgents-ProtoPads" package="EIA-0402" value="10k" x="53.87009375" y="75.058778125" smashed="yes" rot="R180"/>
 <element name="R220" library="PatternAgents-ProtoPads" package="EIA-0402" value="10k" x="57.068465625" y="75.0735125" smashed="yes"/>
 <element name="P201" library="503148-1690" package="MOLEX_503148-1690" value="503148-1690" x="40.344596875" y="74.433678125" smashed="yes">
@@
 <contactref element="C202" pad="2"/>
 <contactref element="R218" pad="2"/>
-<contactref element="R19" pad="2"/>
+<contactref element="R219" pad="2"/>
 <contactref element="R220" pad="2"/>
 <contactref element="P202" pad="4"/>
@@
 <contactref element="U201" pad="2"/>
 <contactref element="SJ2" pad="2"/>
-<contactref element="R19" pad="1"/>
+<contactref element="R219" pad="1"/>
 <wire x1="53.308503125" y1="73.9648" x2="54.483" y2="75.057" width="0.2032" layer="1"/>
 <wire x1="53.307740625" y1="72.8149375" x2="53.308503125" y2="73.9648" width="0.2032" layer="16"/>
