File: MarkIIIB/driver_03_12_2018/driver_03_12_2018.sch (EAGLE design)
At the start: 37 parts, among them P201 503148-1690, P202 502494-0670, U201 PCA9548A_PW_24

Commit message: Add Part Number ROllup Spreadsheets
Parts:
- renumbered R19 to R219
Changed lines of the file:
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@@
 <part name="R217" library="resistor" deviceset="R-US_" device="R0402" value="10k"/>
 <part name="R218" library="PatternAgents-ProtoPads" deviceset="RESISTOR" device="0402-TYP" value="10k"/>
-<part name="R19" library="PatternAgents-ProtoPads" deviceset="RESISTOR" device="0402-TYP" value="10k"/>
+<part name="R219" library="PatternAgents-ProtoPads" deviceset="RESISTOR" device="0402-TYP" value="10k"/>
 <part name="R220" library="PatternAgents-ProtoPads" deviceset="RESISTOR" device="0402-TYP" value="10k"/>
 <part name="P201" library="503148-1690" deviceset="503148-1690" device=""/>
@@
 <instance part="R217" gate="G$1" x="48.26" y="200.66"/>
 <instance part="R218" gate="R" x="231.14" y="129.54" rot="R270"/>
-<instance part="R19" gate="R" x="223.52" y="129.54" rot="R270"/>
+<instance part="R219" gate="R" x="223.52" y="129.54" rot="R270"/>
 <instance part="R220" gate="R" x="215.9" y="129.54" rot="R270"/>
 <instance part="P201" gate="G$1" x="193.04" y="139.7"/>
@@
 <wire x1="223.52" y1="124.46" x2="223.52" y2="119.38" width="0.1524" layer="91"/>
 <label x="223.52" y="119.38" size="1.778" layer="95" rot="R270"/>
-<pinref part="R19" gate="R" pin="2"/>
+<pinref part="R219" gate="R" pin="2"/>
 </segment>
 <segment>
@@
 <wire x1="223.52" y1="142.24" x2="223.52" y2="134.62" width="0.1524" layer="91"/>
 <label x="223.52" y="139.7" size="1.778" layer="95" rot="R270"/>
-<pinref part="R19" gate="R" pin="1"/>
+<pinref part="R219" gate="R" pin="1"/>
 </segment>
 </net>
