File: MarkIIIB/imu_03_12_2018/imu_03_12_2018.sch (EAGLE design)
At the start: 12 parts, among them P301 502585-0470, U301 BNO055

Commit message: Add Part Number ROllup Spreadsheets
Parts:
- C301, C302, C303, C304: device rcl:C-USC0402 -> PatternAgents-ProtoPads:CAP0402-CAP
- R301, R302, R303, R304: device rcl:R-US_R0402 -> PatternAgents-ProtoPads:RESISTOR0402-TYP
Other:
- moved on the sheet: C301, C302, C303, C304
Changed lines of the file:
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@@
 <part name="U301" library="microbuilder" deviceset="BNO055" device="" value="BNO055"/>
 <part name="P301" library="502585-0470" deviceset="502585-0470" device=""/>
-<part name="C302" library="rcl" deviceset="C-US" device="C0402" value="0.1u"/>
-<part name="C303" library="rcl" deviceset="C-US" device="C0402" value="0.1u"/>
+<part name="C302" library="PatternAgents-ProtoPads" deviceset="CAP" device="0402-CAP" value="0.1u"/>
+<part name="C303" library="PatternAgents-ProtoPads" deviceset="CAP" device="0402-CAP" value="0.1u"/>
 <part name="D301" library="led" deviceset="LED" device="CHIP-LED0603"/>
-<part name="R303" library="rcl" deviceset="R-US_" device="R0402" value="220"/>
+<part name="R303" library="PatternAgents-ProtoPads" deviceset="RESISTOR" device="0402-TYP" value="220"/>
 <part name="FRAME1" library="PatternAgents-Beautify" deviceset="FRAME_ASIZE_LANDSCAPE" device=""/>
-<part name="R302" library="rcl" deviceset="R-US_" device="R0402" value="4.7k"/>
-<part name="R301" library="rcl" deviceset="R-US_" device="R0402" value="4.7k"/>
-<part name="C301" library="rcl" deviceset="C-US" device="C0402" value="10uF"/>
+<part name="R302" library="PatternAgents-ProtoPads" deviceset="RESISTOR" device="0402-TYP" value="4.7k"/>
+<part name="R301" library="PatternAgents-ProtoPads" deviceset="RESISTOR" device="0402-TYP" value="4.7k"/>
+<part name="C301" library="PatternAgents-ProtoPads" deviceset="CAP" device="0402-CAP" value="10uF"/>
 <part name="L301" library="halcyonmod_Passives" deviceset="SMD-FERRITE-CHIP-120-OHM-500MA(0603)" device="" value="120OHM-500MA"/>
 <part name="U$2" library="PatternAgents-Beautify" deviceset="GND" device=""/>
 <part name="U$5" library="PatternAgents-Beautify" deviceset="GND" device=""/>
 <part name="U$6" library="PatternAgents-Beautify" deviceset="GND" device=""/>
-<part name="C304" library="rcl" deviceset="C-US" device="C0402" value="0.1u"/>
-<part name="R304" library="rcl" deviceset="R-US_" device="R0402" value="4.7k"/>
+<part name="C304" library="PatternAgents-ProtoPads" deviceset="CAP" device="0402-CAP" value="0.1u"/>
+<part name="R304" library="PatternAgents-ProtoPads" deviceset="RESISTOR" device="0402-TYP" value="4.7k"/>
 <part name="U$8" library="PatternAgents-Beautify" deviceset="GND" device=""/>
 </parts>
@@
 </instance>
 <instance part="D301" gate="G$1" x="106.68" y="101.6" rot="MR0"/>
-<instance part="R303" gate="G$1" x="106.68" y="114.3" rot="MR270"/>
+<instance part="R303" gate="R" x="106.68" y="114.3" rot="MR270"/>
 <instance part="FRAME1" gate="G$2" x="172.72" y="0"/>
 <instance part="FRAME1" gate="G$1" x="0" y="0"/>
-<instance part="R302" gate="G$1" x="121.92" y="139.7" rot="MR270"/>
-<instance part="R301" gate="G$1" x="129.54" y="139.7" rot="MR270"/>
+<instance part="R302" gate="R" x="121.92" y="139.7" rot="MR270"/>
+<instance part="R301" gate="R" x="129.54" y="139.7" rot="MR270"/>
 <instance part="C301" gate="G$1" x="96.52" y="101.6" smashed="yes" rot="MR0">
 <attribute name="NAME" x="89.916" y="95.885" size="1.778" layer="95" rot="MR180"/>
@@
 <attribute name="VALUE" x="117.856" y="98.171" size="1.778" layer="96" rot="MR180"/>
 </instance>
-<instance part="R304" gate="G$1" x="116.84" y="114.3" rot="MR270"/>
+<instance part="R304" gate="R" x="116.84" y="114.3" rot="MR270"/>
 <instance part="U$8" gate="G$1" x="116.84" y="91.44" rot="MR0"/>
 </instances>
@@
 <wire x1="187.96" y1="104.14" x2="182.88" y2="104.14" width="0.1524" layer="91"/>
 <pinref part="C303" gate="G$1" pin="2"/>
-<wire x1="193.04" y1="111.76" x2="193.04" y2="104.14" width="0.1524" layer="91"/>
+<wire x1="193.04" y1="114.3" x2="193.04" y2="104.14" width="0.1524" layer="91"/>
 <wire x1="193.04" y1="104.14" x2="187.96" y2="104.14" width="0.1524" layer="91"/>
 <junction x="187.96" y="104.14"/>
@@
 <pinref part="C302" gate="G$1" pin="2"/>
 <wire x1="193.04" y1="104.14" x2="208.28" y2="104.14" width="0.1524" layer="91"/>
-<wire x1="208.28" y1="104.14" x2="208.28" y2="111.76" width="0.1524" layer="91"/>
+<wire x1="208.28" y1="104.14" x2="208.28" y2="114.3" width="0.1524" layer="91"/>
 <pinref part="U301" gate="G$1" pin="GND@1"/>
 <wire x1="182.88" y1="116.84" x2="187.96" y2="116.84" width="0.1524" layer="91"/>
@@
 <segment>
 <pinref part="C301" gate="G$1" pin="2"/>
-<wire x1="96.52" y1="91.44" x2="96.52" y2="96.52" width="0.1524" layer="91"/>
+<wire x1="96.52" y1="91.44" x2="96.52" y2="99.06" width="0.1524" layer="91"/>
 <pinref part="U$6" gate="G$1" pin="GND"/>
 </segment>
@@
 <pinref part="U$8" gate="G$1" pin="GND"/>
 <pinref part="C304" gate="G$1" pin="2"/>
-<wire x1="116.84" y1="96.52" x2="116.84" y2="91.44" width="0.1524" layer="91"/>
+<wire x1="116.84" y1="99.06" x2="116.84" y2="91.44" width="0.1524" layer="91"/>
 </segment>
 </net>
@@
 <wire x1="195.58" y1="121.92" x2="193.04" y2="121.92" width="0.1524" layer="91"/>
 <wire x1="193.04" y1="121.92" x2="182.88" y2="121.92" width="0.1524" layer="91"/>
-<wire x1="193.04" y1="119.38" x2="193.04" y2="121.92" width="0.1524" layer="91"/>
 <junction x="193.04" y="121.92"/>
 </segment>
@@
 <pinref part="U301" gate="G$1" pin="COM0/SDA/TX"/>
 <label x="137.16" y="129.54" size="1.778" layer="95" rot="MR0"/>
-<pinref part="R301" gate="G$1" pin="2"/>
+<pinref part="R301" gate="R" pin="2"/>
 <wire x1="142.24" y1="129.54" x2="129.54" y2="129.54" width="0.1524" layer="91"/>
 <wire x1="129.54" y1="129.54" x2="129.54" y2="134.62" width="0.1524" layer="91"/>
@@
 <pinref part="U301" gate="G$1" pin="COM1/SCL/RX"/>
 <label x="137.16" y="127" size="1.778" layer="95" rot="MR0"/>
-<pinref part="R302" gate="G$1" pin="2"/>
+<pinref part="R302" gate="R" pin="2"/>
 <wire x1="142.24" y1="127" x2="121.92" y2="127" width="0.1524" layer="91"/>
 <wire x1="121.92" y1="127" x2="121.92" y2="134.62" width="0.1524" layer="91"/>
@@
 <net name="N$2" class="0">
 <segment>
-<pinref part="R303" gate="G$1" pin="2"/>
+<pinref part="R303" gate="R" pin="2"/>
 <pinref part="D301" gate="G$1" pin="A"/>
 <wire x1="106.68" y1="109.22" x2="106.68" y2="104.14" width="0.1524" layer="91"/>
@@
 <pinref part="C302" gate="G$1" pin="1"/>
 <wire x1="182.88" y1="127" x2="208.28" y2="127" width="0.1524" layer="91"/>
-<wire x1="208.28" y1="127" x2="208.28" y2="119.38" width="0.1524" layer="91"/>
+<wire x1="208.28" y1="127" x2="208.28" y2="121.92" width="0.1524" layer="91"/>
 <pinref part="U301" gate="G$1" pin="VDD"/>
 <wire x1="182.88" y1="129.54" x2="208.28" y2="129.54" width="0.1524" layer="91"/>
@@
 <wire x1="106.68" y1="149.86" x2="106.68" y2="119.38" width="0.1524" layer="91"/>
 <pinref part="L301" gate="L" pin="1"/>
-<pinref part="R302" gate="G$1" pin="1"/>
+<pinref part="R302" gate="R" pin="1"/>
 <wire x1="96.52" y1="121.92" x2="91.44" y2="121.92" width="0.1524" layer="91"/>
 <wire x1="121.92" y1="144.78" x2="121.92" y2="149.86" width="0.1524" layer="91"/>
 <junction x="121.92" y="149.86"/>
-<pinref part="R301" gate="G$1" pin="1"/>
+<pinref part="R301" gate="R" pin="1"/>
 <wire x1="129.54" y1="144.78" x2="129.54" y2="149.86" width="0.1524" layer="91"/>
 <junction x="129.54" y="149.86"/>
-<pinref part="R303" gate="G$1" pin="1"/>
+<pinref part="R303" gate="R" pin="1"/>
 <label x="210.82" y="149.86" size="1.27" layer="95" font="vector" ratio="10" rot="MR180" xref="yes"/>
 <wire x1="106.68" y1="149.86" x2="96.52" y2="149.86" width="0.1524" layer="91"/>
 <junction x="106.68" y="149.86"/>
-<pinref part="R304" gate="G$1" pin="1"/>
+<pinref part="R304" gate="R" pin="1"/>
 <wire x1="116.84" y1="119.38" x2="116.84" y2="149.86" width="0.1524" layer="91"/>
 <junction x="116.84" y="149.86"/>
 <pinref part="C301" gate="G$1" pin="1"/>
-<wire x1="96.52" y1="104.14" x2="96.52" y2="121.92" width="0.1524" layer="91"/>
+<wire x1="96.52" y1="106.68" x2="96.52" y2="121.92" width="0.1524" layer="91"/>
 <junction x="96.52" y="121.92"/>
 <wire x1="96.52" y1="121.92" x2="96.52" y2="149.86" width="0.1524" layer="91"/>
@@
 <net name="!RST" class="0">
 <segment>
-<pinref part="R304" gate="G$1" pin="2"/>
+<pinref part="R304" gate="R" pin="2"/>
 <pinref part="C304" gate="G$1" pin="1"/>
 <wire x1="116.84" y1="109.22" x2="116.84" y2="106.68" width="0.1524" layer="91"/>
 <pinref part="U301" gate="G$1" pin="NRESET"/>
-<wire x1="116.84" y1="106.68" x2="116.84" y2="104.14" width="0.1524" layer="91"/>
 <wire x1="142.24" y1="111.76" x2="132.08" y2="111.76" width="0.1524" layer="91"/>
 <wire x1="132.08" y1="111.76" x2="132.08" y2="106.68" width="0.1524" layer="91"/>
