File: MarkIIIB/imu_b_03_12_2018/imu_b_03_12_2018.brd (EAGLE design)
At the start: 16 x 19.9 mm, 15 parts, among them P401 502585-0470, U401 BNO055

Commit message: Add Part Number ROllup Spreadsheets
Parts:
- C401, C402, C403, C404: device rcl:C0402 -> PatternAgents-ProtoPads:0402-CAP
- R401, R402, R403, R404: device rcl:R0402 -> PatternAgents-ProtoPads:EIA-0402
Routing:
- net GND: track 28.4 -> 29.2 mm
- net VDD: track 30.9 -> 31.5 mm
